File: Remote-ZIF42/Remote-ZIF42.kicad_pcb (KiCad board)
At the start: 2 copper layers, 82.2 x 52.1 mm, 23 parts, among them J1 ZIF-48, J2 EXTRA, J3 IDC-10, J4 IDC-40, J5 FFC-50, J6 SHIELD, SW1 RESET

Commit message: Remote-ZIF42 v1.1 enlarge through-holes for socket, cleanup routing
Parts:
- moved SW1 5.68 mm to (42.6, 22.1)
- moved J5 5.68 mm to (70.5, 63.1)
- moved D1 5.68 mm to (94.0, 19.7)
- moved C1 5.68 mm to (97.8, 21.6)
- moved H1 5.68 mm to (29.1, 19.6)
- moved H2 5.68 mm to (104.1, 19.6)
- moved J1 5.68 mm to (40.6, 43.2)
- moved J2 5.68 mm to (67.3, 21.6)
- moved J3 5.68 mm to (31.8, 54.6)
- moved J4 5.68 mm to (53.3, 54.6)
- moved JP1 5.68 mm to (78.7, 21.6)
- moved R2 5.68 mm to (94.0, 22.2)
- moved H3 5.68 mm to (29.1, 64.5)
- moved H4 5.68 mm to (104.1, 64.5)
- moved J6 5.68 mm to (88.9, 64.1)
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Routing:
- net /A17: track 70.5 -> 52.2 mm, vias 2 -> 1
- net /A16: track 87.0 -> 94.3 mm, vias 2 -> 0
- net /A19: track 74.8 -> 75.9 mm
- net /A13: track 35.5 -> 36.5 mm
- net /A12: track 36.1 -> 37.2 mm
- net /A9: track 39.5 -> 40.5 mm
- net /A8: track 41.0 -> 42.0 mm
- net /A11: track 36.8 -> 37.8 mm
- net /A10: track 37.9 -> 39.0 mm
- net /A15: track 35.6 -> 36.6 mm
- net /A14: track 35.0 -> 36.0 mm
